Commit message: Add files via upload

File: urdf/efectorfinal.urdf (robot description, URDF)
Before this commit: robot efectorfinal, 4 links, 3 joints
Joints:
- joint first_joint: limit (none) -> lower=0 upper=0 effort=0 velocity=0; origin xyz=0 0 0 rpy=1.70031185920797 0 -1.5707963267949 -> xyz=0 0 0 rpy=1.7003 0 -1.5708; type continuous -> revolute
- joint second_joint: axis 0 0 0 -> 1 0 0; type fixed -> continuous
- joint third_joint: axis 0 0 0 -> 1 0 0; origin xyz=0.01 0.014838 -0.03319 rpy=1.5708 -1.4413 1.5708 -> xyz=0.01 0.0148375966439305 -0.0331904766116383 rpy=1.5707963267949 -1.44128079438183 1.5707963267949; type fixed -> continuous

Commit message: Add files via upload

File: urdf/efectorfinal.urdf (robot description, URDF)
Before this commit: robot efectorfinal, 4 links, 3 joints
Links:
- link base_link: mass 0.162356194490192 -> 0.16236
- link first_Link: mass 0.00618813972610106 -> 0.0061881
- link second_link: mass 0.0103535967073896 -> 0.010354
- link third_link: mass 0.0103535967081163 -> 0.010354
Joints:
- joint first_joint: origin xyz=0 0 0 rpy=1.7003 0 -1.5708 -> xyz=0 0.048 0.08 rpy=-1.3749 0 1.5708
- joint second_joint: axis 1 0 0 -> 0 0 0; limit (none) -> lower=0 upper=0 effort=0 velocity=0; origin xyz=0.01 -0.0148310357596693 0.0332408501719503 rpy=-1.5707963267949 1.44128079438183 -1.5707963267949 -> xyz=0.01 -0.012796 0.033125 rpy=-1.5708 1.3749 -1.5708; type continuous -> prismatic
- joint third_joint: axis 1 0 0 -> 0 0 0; limit (none) -> lower=0 upper=0 effort=0 velocity=0; origin xyz=0.01 0.0148375966439305 -0.0331904766116383 rpy=1.5707963267949 -1.44128079438183 1.5707963267949 -> xyz=0.01 0.012796 -0.033125 rpy=1.5708 -1.3749 1.5708; type continuous -> prismatic

Commit message: Add files via upload

File: urdf/efectorfinal.urdf (robot description, URDF)
Before this commit: robot efectorfinal, 4 links, 3 joints
Links:
- removed link first_Link
- removed link third_link
- added link first_link, mass 0.010354; collision mesh filename=package://efectorfinal/meshes/first_link.STL; visual mesh filename=package://efectorfinal/meshes/first_link.STL
- link base_link: mass 0.16236 -> 0.16854
Joints:
- removed joint third_joint
- joint first_joint: axis -1 0 0 -> 0 0 0; child first_Link -> first_link; limit lower=0 upper=0 effort=0 velocity=0 -> lower=-0.02 upper=0.02 effort=0 velocity=0; origin xyz=0 0.048 0.08 rpy=-1.3749 0 1.5708 -> xyz=-0.03 0.058 0.099 rpy=-1.5708 0 0; type revolute -> prismatic
- joint second_joint: limit lower=0 upper=0 effort=0 velocity=0 -> lower=-0.02 upper=0.02 effort=0 velocity=0; origin xyz=0.01 -0.012796 0.033125 rpy=-1.5708 1.3749 -1.5708 -> xyz=0.03 0.058 0.061 rpy=1.5708 0 -3.1416; parent first_Link -> base_link
